Commit message: Adjusted wheel collisions

File: urdf/dalek.urdf (robot description, URDF)
Before this commit: robot dalek, 5 links, 4 joints
Links:
- link front_wheel: mass 0.4 -> 1
- link left_back_wheel: mass 0.4 -> 1
- link right_back_wheel: mass 0.4 -> 1
Joints:
- removed joint base_to_head
- added joint head_swivel: type continuous, parent base_link, child head, origin xyz=0 0 0.3, axis 0 0 1

Commit message: Corrected head position

File: urdf/dalek.urdf (robot description, URDF)
Before this commit: robot dalek, 5 links, 4 joints
Joints:
- joint front_wheel_joint: type fixed -> continuous
- joint head_swivel: origin xyz=0 0 0.3 -> xyz=0 0 0

Commit message: Joint parameters updated for head

File: urdf/dalek.urdf (robot description, URDF)
Before this commit: robot dalek, 5 links, 4 joints
Joints:
- joint head_swivel: limit (none) -> effort=30 velocity=1.0
